File: hardware/board_v0.0.1/_autosave-shield_v0.0.1.kicad_sch (KiCad schematic)
At the start: 17 parts, among them IC1 BQ25172DSGR, IC2 TPS2117DRLR, J1 USB_C_Receptacle_PowerOnly_6P, U1 STM32L053R8Tx

Commit message: Added extra components
Parts:
- added C3: 1u, symbol Device:C
- added C4, C5, C6, C7: 100n, symbol Device:C
- added U2: nRF24L01P, Package_DFN_QFN:QFN-20-1EP_4x4mm_P0.5mm_EP2.5x2.5mm, symbol RF:nRF24L01P
- R8, R9: value 18k -> 1k
Connections:
- net GND: now also C3.2, C4.2, C5.2, C6.2, C7.2
- net +3.3V: now reaches U1.13 (VDDA)
- net +3.3V: now also U1.19 (VDD), U1.32 (VDD), U1.64 (VDD), C3.1, C4.1, C5.1, C6.1, C7.1
Other:
- moved on the sheet: BT1, C1, C2, D1, IC1, IC2, J1, R1, R2, R3, R4, R5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
